Commit message: Temp_analise_use

File: ws/src/agv/agv_description/urdf/agv_base.urdf.xacro (robot description, xacro)
@@ -101,9 +101,9 @@
       <parent link="base_link"/>
       <child link="zed_camera"/>
-      <origin xyz="0.49 0 0.175" rpy="0 0 0" />
+      <origin xyz="0.90 0 0.175" rpy="0 1.57 0" />
     </joint>
     <gazebo reference="zed_camera">
       <sensor type="camera" name="camera">
-        <update_rate>30.0</update_rate>
+        <update_rate>100.0</update_rate>
         <camera name="head">
           <horizontal_fov>1.3962634</horizontal_fov>
@@ -128,5 +128,5 @@
         <plugin name="camera_controller" filename="libgazebo_ros_camera.so">
           <alwaysOn>true</alwaysOn>
-          <updateRate>0.0</updateRate>
+          <updateRate>500</updateRate>
           <cameraName>camera</cameraName>
           <imageTopicName>image_raw</imageTopicName>
