Commit message: Changed position of camera in robot

File: src/agv/agv_description/urdf/agv_base.urdf.xacro (robot description, xacro)
@@ -7,5 +7,6 @@
         <origin xyz="0 0 -0.1625" rpy=" 0 0 0"/>
         <geometry>
-          <mesh filename="package://agv_description/meshes/OTAv07_meshes/OTA-v0.7.stl" scale="0.001 0.001 0.001"/>
+           <!--<mesh filename="package://agv_description/meshes/OTAv07_meshes/OTA-v0.7.stl" scale="0.001 0.001 0.001"/> -->
+          <box size="1.02 0.72 0.14"/>
         </geometry>
       </visual>
@@ -101,9 +102,9 @@
       <parent link="base_link"/>
       <child link="zed_camera"/>
-      <origin xyz="0.49 0 0.175" rpy="0 0 0" />
+            <origin xyz="0.90 0 0.175" rpy="0 1.57 0" />
     </joint>
     <gazebo reference="zed_camera">
       <sensor type="camera" name="camera">
-        <update_rate>30.0</update_rate>
+        <update_rate>100.0</update_rate>
         <camera name="head">
           <horizontal_fov>1.3962634</horizontal_fov>
@@ -128,5 +129,5 @@
         <plugin name="camera_controller" filename="libgazebo_ros_camera.so">
           <alwaysOn>true</alwaysOn>
-          <updateRate>0.0</updateRate>
+          <updateRate>500.0</updateRate>
           <cameraName>camera</cameraName>
           <imageTopicName>image_raw</imageTopicName>

Commit message: Melhoria no modelo do robô para exibição no RVIZ

File: src/agv/agv_description/urdf/agv_base.urdf.xacro (robot description, xacro)
@@ -8,5 +8,5 @@
         <geometry>
            <!--<mesh filename="package://agv_description/meshes/OTAv07_meshes/OTA-v0.7.stl" scale="0.001 0.001 0.001"/> -->
-          <box size="1.02 0.72 0.14"/>
+          <box size="1.02 0.72 0.40"/>
         </geometry>
       </visual>
